File: BLDC_controller.kicad_pcb (KiCad board)
At the start: 4 copper layers, 50 x 38 mm, 371 parts, among them P2 CONN_01X06, P3 CONN_01X05, P5 CONN_01X05, Q1 PSMN2R0-30YLD, Q2 PSMN2R0-30YLD, Q3 PSMN2R0-30YLD, Q4 PSMN2R0-30YLD, Q5 PSMN2R0-30YLD, Q6 PSMN2R0-30YLD

Commit message: firts review comments updated
Parts:
- removed the REF** at (172.5, 87.5)
- removed the REF** at (172.5, 92.5)
- removed the REF** at (172.5, 98.3)
- removed the REF** at (173.0, 107.0)
- added REF**: VIA-0.8mm-0.4mm, project_footprints:VIA-0.8mm-0.4mm, F.Cu at (178.7, 109.9)
- added REF**: VIA-0.8mm-0.4mm, project_footprints:VIA-0.8mm-0.4mm, F.Cu at (173.1, 109.2)
- added REF**: VIA-0.8mm-0.4mm, project_footprints:VIA-0.8mm-0.4mm, F.Cu at (146.0, 98.3)
- added REF***: OSHW-Logo2_7.3x6mm_SilkScreen, Symbols:OSHW-Logo2_7.3x6mm_SilkScreen, F.Cu at (139.9, 90.6)
- moved REF** 1.25 mm to (173.0, 82.0)
- moved REF** 0.98 mm to (172.2, 91.2)
- moved V5 0.46 mm to (159.8, 80.9)
- moved C7 0.45 mm to (145.2, 108.2)
- moved V1 0.41 mm to (150.0, 106.5)
- moved L1 0.35 mm to (144.9, 104.8)
- moved C4 0.25 mm to (176.0, 82.2)
- moved C16 0.19 mm to (150.3, 91.3)
- moved REF** 0.10 mm to (183.1, 95.7)
- moved REF** 0.10 mm to (183.1, 91.6)
- moved REF** 0.10 mm to (183.1, 90.9)
- moved REF** 0.10 mm to (183.1, 90.2)
- moved REF** 0.10 mm to (183.1, 89.5)
- moved REF** 0.10 mm to (183.1, 88.8)
- moved REF** 0.10 mm to (183.1, 88.1)
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Routing:
- net +12V: track 37.9 -> 62.5 mm, vias 12 -> 11
- net GND: track 115.8 -> 124.4 mm, vias 27 -> 28
- net V_SENSE_P: track 7.63 -> 15.2 mm
- net U_SENSE_P: track 12.9 -> 19.8 mm
- net W_SENSE_P: track 12.2 -> 19.1 mm
- net +3V3: track 30.0 -> 28.0 mm
- net Net-(R40-Pad2): track 0.00 -> 1.41 mm
- net /OUTV: track 33.8 -> 35.0 mm
- net /HSW: track 18.2 -> 17.2 mm
- net /NRST: track 36.9 -> 37.9 mm
- net /HSU: track 25.2 -> 26.0 mm
- net /OUTW: track 36.6 -> 37.4 mm
- net /HALL1/A+: track 28.5 -> 29.2 mm
- net /V_ADC: track 21.7 -> 22.4 mm
- net Net-(D1-Pad36): track 15.7 -> 16.3 mm
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- added copper zone on In1.Cu, net /OUTU
- added copper zone on In1.Cu, net /OUTV
- added copper zone on In1.Cu, net /OUTW
Other:
- board text added: "+12V"
- board text added: "+3.3V"
- board text added: "GND"
- board text added: "HALL1"
- board text added: "HALL2"
- board text added: "HALL3"
- board text added: "MISO"
- board text added: "MOSI"
- board text added: "NSS"
- board text added: "SCK"
- board text added: "ST-LINK"

Commit message: minor corrections
Other:
- rule pad_to_mask_clearance: 0.2 -> 0.075
Changed lines of the file:
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@@
     (links 554)
     (no_connects 94)
-    (area 135.174999 77.929999 185.325001 116.080001)
+    (area 135.174999 77.924999 185.325001 116.080001)
     (thickness 1.6)
-    (drawings 34)
+    (drawings 36)
     (tracks 977)
     (zones 0)
@@
     (1 In1.Cu power hide)
     (2 In2.Cu power hide)
-    (31 B.Cu signal hide)
-    (32 B.Adhes user hide)
-    (33 F.Adhes user hide)
-    (34 B.Paste user hide)
-    (35 F.Paste user hide)
-    (36 B.SilkS user hide)
+    (31 B.Cu signal)
+    (32 B.Adhes user)
+    (33 F.Adhes user)
+    (34 B.Paste user)
+    (35 F.Paste user)
+    (36 B.SilkS user)
     (37 F.SilkS user)
     (38 B.Mask user)
-    (39 F.Mask user hide)
+    (39 F.Mask user)
     (40 Dwgs.User user)
     (41 Cmts.User user)
@@
     (pad_size 1.35 1.55)
     (pad_drill 0)
-    (pad_to_mask_clearance 0.2)
+    (pad_to_mask_clearance 0.075)
     (solder_mask_min_width 0.1)
-    (aux_axis_origin 135.25 116.005)
-    (visible_elements FFFFFF7F)
+    (pad_to_paste_clearance -0.05)
+    (aux_axis_origin 135.25 116)
+    (grid_origin 135.25 116)
+    (visible_elements FFFF7F7F)
     (pcbplotparams
-      (layerselection 0x000fc_80000007)
-      (usegerberextensions false)
+      (layerselection 0x018fc_80000007)
+      (usegerberextensions true)
       (excludeedgelayer true)
       (linewidth 0.100000)
-      (plotframeref true)
+      (plotframeref false)
       (viasonmask false)
       (mode 1)
@@
     (tags "capacitor 0603")
     (attr smd)
-    (fp_text reference C1 (at 0.85 1.45 180) (layer F.SilkS)
+    (fp_text reference C1 (at 2.08 0.01 180) (layer F.SilkS)
       (effects (font (size 0.8 0.8) (thickness 0.15)))
     )
@@
     (tags "resistor 2512")
     (attr smd)
-    (fp_text reference R7 (at 1.05 -3.1 360) (layer B.SilkS)
+    (fp_text reference R7 (at 3.835 -2.97 360) (layer B.SilkS)
       (effects (font (size 1 1) (thickness 0.15)) (justify mirror))
     )
@@
     (tags "resistor 2512")
     (attr smd)
-    (fp_text reference R8 (at -3.9 -3.75 360) (layer B.SilkS)
+    (fp_text reference R8 (at -4.605 -0.05 360) (layer B.SilkS)
       (effects (font (size 1 1) (thickness 0.15)) (justify mirror))
     )
@@
   )
   (module Connect:1pin (layer F.Cu)
-    (at 138.5 81.255)
+    (at 138.5 81.25)
     (descr "module 1 pin (ou trou mecanique de percage)")
     (tags DEV)
@@
   )
   (module Connect:1pin (layer F.Cu)
-    (at 138.5 112.755)
+    (at 138.5 112.75)
     (descr "module 1 pin (ou trou mecanique de percage)")
     (tags DEV)
@@
     (tags "LFPAK SOT-669 Power-SO8")
     (attr smd)
-    (fp_text reference Q2 (at 3.595 1.35 180) (layer B.SilkS)
+    (fp_text reference Q2 (at 3.49 2.24 180) (layer B.SilkS)
       (effects (font (size 0.8 0.8) (thickness 0.15)) (justify mirror))
     )
@@
     (tags "LFPAK SOT-669 Power-SO8")
     (attr smd)
-    (fp_text reference Q4 (at 3.6 2.9 180) (layer B.SilkS)
+    (fp_text reference Q4 (at 3.615 3.14 180) (layer B.SilkS)
       (effects (font (size 0.8 0.8) (thickness 0.15)) (justify mirror))
     )
@@
     (tags SOD-323)
     (attr smd)
-    (fp_text reference V2 (at 0.65 -1.7 180) (layer F.SilkS)
+    (fp_text reference V2 (at 2.3 -0.65 180) (layer F.SilkS)
       (effects (font (size 0.8 0.8) (thickness 0.15)))
     )
@@
     (tags "resistor 2512")
     (attr smd)
-    (fp_text reference R9 (at 2.795 2.85 180) (layer B.SilkS)
+    (fp_text reference R9 (at 2.7 2.81 180) (layer B.SilkS)
       (effects (font (size 0.8 0.8) (thickness 0.15)) (justify mirror))
     )
@@
     (tags "capacitor 0805")
     (attr smd)
-    (fp_text reference C17 (at -3.7 -4.15 360) (layer F.SilkS)
+    (fp_text reference C17 (at -3.64 -4.17 360) (layer F.SilkS)
       (effects (font (size 0.8 0.8) (thickness 0.15)))
     )
@@
     (tags "capacitor 0603")
     (attr smd)
-    (fp_text reference C14 (at -2 0.1 360) (layer F.SilkS)
+    (fp_text reference C14 (at -2.05 0.27 360) (layer F.SilkS)
       (effects (font (size 0.8 0.8) (thickness 0.15)))
     )
@@
     (tags "resistor 0603")
     (attr smd)
-    (fp_text reference R35 (at -2.5 0.195 180) (layer B.SilkS)
+    (fp_text reference R35 (at -2.48 0.23 180) (layer B.SilkS)
       (effects (font (size 0.8 0.8) (thickness 0.15)) (justify mirror))
     )
@@
     (tags "resistor 0603")
     (attr smd)
-    (fp_text reference R22 (at -2.8 -0.075 360) (layer B.SilkS)
+    (fp_text reference R22 (at -1.57 -1.365 360) (layer B.SilkS)
       (effects (font (size 0.8 0.8) (thickness 0.15)) (justify mirror))
     )
@@
     (tags "resistor 0603")
     (attr smd)
-    (fp_text reference R42 (at 2 1.095 180) (layer B.SilkS)
+    (fp_text reference R42 (at 2.03 1.05 180) (layer B.SilkS)
       (effects (font (size 0.8 0.8) (thickness 0.15)) (justify mirror))
     )
@@
     (tags "resistor 0603")
     (attr smd)
-    (fp_text reference R45 (at 4.1 1.1) (layer B.SilkS)
+    (fp_text reference R45 (at 4.22 1.14) (layer B.SilkS)
       (effects (font (size 0.8 0.8) (thickness 0.15)) (justify mirror))
     )
@@
     (tags "resistor 0603")
     (attr smd)
-    (fp_text reference R37 (at -0.05 1.15 180) (layer F.SilkS)
+    (fp_text reference R37 (at 0.05 1.2 180) (layer F.SilkS)
       (effects (font (size 0.8 0.8) (thickness 0.15)))
     )
@@
     (tags "QFN 0.5")
     (attr smd)
-    (fp_text reference D1 (at 0 -4.75) (layer F.SilkS)
+    (fp_text reference D1 (at 0.71 -4.815) (layer F.SilkS)
       (effects (font (size 0.8 0.8) (thickness 0.15)))
     )
@@
     )
   )
+  (dimension 38 (width 0.3) (layer Eco2.User)
+    (gr_text "38,000 mm" (at 196.6 97 270) (layer Eco2.User)
+      (effects (font (size 1.5 1.5) (thickness 0.3)))
+    )
+    (feature1 (pts (xy 185.25 116) (xy 197.95 116)))
+    (feature2 (pts (xy 185.25 78) (xy 197.95 78)))
+    (crossbar (pts (xy 195.25 78) (xy 195.25 116)))
+    (arrow1a (pts (xy 195.25 116) (xy 194.663579 114.873496)))
+    (arrow1b (pts (xy 195.25 116) (xy 195.836421 114.873496)))
+    (arrow2a (pts (xy 195.25 78) (xy 194.663579 79.126504)))
+    (arrow2b (pts (xy 195.25 78) (xy 195.836421 79.126504)))
+  )
+  (dimension 50 (width 0.3) (layer Eco2.User)
+    (gr_text "50,000 mm" (at 160.25 68.65) (layer Eco2.User)
+      (effects (font (size 1.5 1.5) (thickness 0.3)))
+    )
+    (feature1 (pts (xy 185.25 78) (xy 185.25 67.3)))
+    (feature2 (pts (xy 135.25 78) (xy 135.25 67.3)))
+    (crossbar (pts (xy 135.25 70) (xy 185.25 70)))
+    (arrow1a (pts (xy 185.25 70) (xy 184.123496 70.586421)))
+    (arrow1b (pts (xy 185.25 70) (xy 184.123496 69.413579)))
+    (arrow2a (pts (xy 135.25 70) (xy 136.376504 70.586421)))
+    (arrow2b (pts (xy 135.25 70) (xy 136.376504 69.413579)))
+  )
   (gr_text GND (at 157.5 109.5 90) (layer F.SilkS)
     (effects (font (size 0.8 0.8) (thickness 0.15)))
@@
     (effects (font (size 0.8 0.8) (thickness 0.15)))
   )
-  (gr_line (start 135.25 116.005) (end 135.25 78.005) (angle 90) (layer Edge.Cuts) (width 0.15))
-  (gr_line (start 185.25 116.005) (end 135.25 116.005) (angle 90) (layer Edge.Cuts) (width 0.15))
-  (gr_line (start 185.25 78.005) (end 185.25 116.005) (angle 90) (layer Edge.Cuts) (width 0.15))
-  (gr_line (start 135.25 78.005) (end 185.25 78.005) (angle 90) (layer Edge.Cuts) (width 0.15))
+  (gr_line (start 135.25 116) (end 135.25 78) (angle 90) (layer Edge.Cuts) (width 0.15))
+  (gr_line (start 185.25 116) (end 135.25 116.005) (angle 90) (layer Edge.Cuts) (width 0.15))
+  (gr_line (start 185.25 78) (end 185.25 116) (angle 90) (layer Edge.Cuts) (width 0.15))
+  (gr_line (start 135.25 78) (end 185.25 78) (angle 90) (layer Edge.Cuts) (width 0.15))
   (via (at 154 107.25) (size 0.8) (drill 0.4) (layers F.Cu B.Cu) (net 0))
   (via (at 152.5 107.25) (size 0.8) (drill 0.4) (layers F.Cu B.Cu) (net 0))
@@
     (polygon
       (pts
-        (xy 135.25 78.005) (xy 178.45 78.005) (xy 178.45 84.705) (xy 168.15 84.705) (xy 168.15 90.755)
+        (xy 135.25 78) (xy 178.5 78) (xy 178.45 84.705) (xy 168.15 84.705) (xy 168.15 90.755)
         (xy 178.35 90.755) (xy 178.45 90.855) (xy 178.45 94.005) (xy 178.35 94.105) (xy 173.65 94.105)
         (xy 173.55 94.003908) (xy 173.55 92.805) (xy 173.35 92.605) (xy 168.15 92.605) (xy 168.15 98.605)
         (xy 171.65 98.605) (xy 173.15 99.705) (xy 178.45 99.705) (xy 178.45 103.005) (xy 173.35 103.005)
         (xy 173 103.255) (xy 171.45 104.405) (xy 168.45 104.405) (xy 168.45 110.305) (xy 172.05 110.305)
-        (xy 172.35 108.505) (xy 178.45 108.505) (xy 178.45 116.005) (xy 135.25 116.005)
+        (xy 172.35 108.505) (xy 178.45 108.505) (xy 178.5 116) (xy 135.25 116)
       )
     )
@@
     (polygon
       (pts
-        (xy 178.5 78.005) (xy 178.5 116.005) (xy 173.5 116.005) (xy 173.5 112.255) (xy 171.5 111.255)
+        (xy 178.5 78) (xy 178.5 116) (xy 173.5 116) (xy 173.5 112.255) (xy 171.5 111.255)
         (xy 171.5 105.005) (xy 172 104.505) (xy 172 100.505) (xy 171.5 100.005) (xy 171.5 83.005)
-        (xy 172.25 82.505) (xy 172.25 78.005)
+        (xy 172.25 82.505) (xy 172.25 78)
       )
     )
@@
       (pts
         (xy 171 100.255) (xy 171.5 100.755) (xy 171.5 104.255) (xy 171 104.755) (xy 171 105.255)
-        (xy 171 111.755) (xy 173 112.755) (xy 173 116.005) (xy 135.25 116.005) (xy 135.25 78.005)
-        (xy 171.75 78.005) (xy 171.75 82.005) (xy 171 82.586341)
+        (xy 171 111.755) (xy 173 112.755) (xy 173 116) (xy 135.25 116) (xy 135.25 78)
+        (xy 171.75 78) (xy 171.75 82.005) (xy 171 82.586341)
       )
     )
